Commit message: Hotfix

File: install/my_robot_description/share/my_robot_description/urdf/my_robot.urdf (robot description, URDF)
Before this commit: robot my_robot, 1 links, 0 joints
Links:
- added link lidar; visual cylinder length=0.05 radius=0.1
Joints:
- added joint base_lidar_joint: type fixed, parent base_link, child lidar, origin xyz=0 0 0 rpy=0 0 0

File: src/my_robot_description/urdf/my_robot.urdf (robot description, URDF)
Before this commit: robot my_robot, 2 links, 1 joints
Links:
- added link base_footprint
- added link caster_wheel; visual sphere radius=0.05
- added link left_wheel; visual cylinder length=0.05 radius=0.1
- added link right_wheel; visual cylinder length=0.05 radius=0.1
Joints:
- added joint base_caster_wheel_joint: type fixed, parent base_link, child caster_wheel, origin xyz=0.2 0 -0.05 rpy=0 0 0
- added joint base_joint: type fixed, parent base_footprint, child base_link, origin xyz=0 0 0.1 rpy=0 0 0
- added joint base_left_wheel_joint: type continuous, parent base_link, child left_wheel, origin xyz=-0.15 0.225 0 rpy=0 0 0, axis 0 1 0
- added joint base_right_wheel_joint: type continuous, parent base_link, child right_wheel, origin xyz=-0.15 -0.225 0 rpy=0 0 0, axis 1 0 0
- joint base_lidar_joint: origin xyz=0 0 0 rpy=0 0 0 -> xyz=0 0 0.225 rpy=0 0 0

Commit message: changes

File: install/my_robot_description/share/my_robot_description/urdf/my_robot.urdf (robot description, URDF)
Before this commit: robot my_robot, 2 links, 1 joints
Links:
- added link base_footprint
- added link caster_wheel; visual sphere radius=0.05
- added link left_wheel; visual cylinder length=0.05 radius=0.1
- added link right_wheel; visual cylinder length=0.05 radius=0.1
Joints:
- added joint base_caster_wheel_joint: type fixed, parent base_link, child caster_wheel, origin xyz=0.2 0 -0.05 rpy=0 0 0
- added joint base_joint: type fixed, parent base_footprint, child base_link, origin xyz=0 0 0.1 rpy=0 0 0
- added joint base_left_wheel_joint: type continuous, parent base_link, child left_wheel, origin xyz=-0.15 0.225 0 rpy=0 0 0, axis 0 1 0
- added joint base_right_wheel_joint: type continuous, parent base_link, child right_wheel, origin xyz=-0.15 -0.225 0 rpy=0 0 0, axis 1 0 0
- joint base_lidar_joint: origin xyz=0 0 0 rpy=0 0 0 -> xyz=0 0 0.225 rpy=0 0 0
